File: dual-vca-kosmo/dual-vca-kosmo.kicad_pcb (KiCad board)
At the start: 2 copper layers, 204 x 200 mm, 94 parts, among them J1 Conn_02x05_Odd_Even, J10 in2, J11 Conn_02x05_Odd_Even, J2 Conn_02x05_Odd_Even, J3 cv1, J4 cv2, J5 cvdual, J6 mixout, J7 out1, J8 out2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

Commit message: Actually update schematic to V1.0
Parts:
- removed R21, R22: 100k, omat:Omaresistor2
- R17, R20: value 47k -> 100k
Connections:
- U3 pad 13: Net-(U3B-IO2) -> Net-(U1A--)
- U3 pad 2: Net-(U3A-IO1) -> Net-(U2D--)
Routing:
- net Net-(U1A--): track 5.09 -> 45.4 mm
- net Net-(U2D--): track 5.07 -> 39.8 mm
- net Net-(U3B-IO2): track 34.1 -> 0.00 mm
- net Net-(U3A-IO1): track 28.6 -> 0.00 mm

Commit message: Schematic V1.1, fixed CV limiting
Parts:
- R11, R13: value 100k -> 120k
- R42, R43: value 10k -> 22k
Connections:
- R7 pad 1: Net-(R42-Pad2) -> Net-(D5-A)
- R8 pad 1: Net-(R43-Pad2) -> Net-(D6-A)
Routing:
- net Net-(D6-A): track 2.90 -> 24.0 mm
- net Net-(D5-A): track 3.79 -> 23.4 mm
- net Net-(R42-Pad2): track 12.8 -> 8.79 mm
- net Net-(R43-Pad2): track 13.2 -> 9.78 mm
Changed lines of the file:
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@@
       (stroke (width 0.05) (type solid)) (layer "F.CrtYd"))
     (pad "1" thru_hole circle (at 0 0 270) (size 1.4 1.4) (drill 0.7) (layers "*.Cu" "*.Mask")
-      (net 28 "Net-(R42-Pad2)") (pintype "passive"))
+      (net 13 "Net-(D5-A)") (pintype "passive"))
     (pad "2" thru_hole oval (at 7.62 0 270) (size 1.4 1.4) (drill 0.7) (layers "*.Cu" "*.Mask")
       (net 34 "Net-(U1C--)") (pintype "passive"))
@@
         (effects (font (size 0.5 0.5) (thickness 0.125)))
     )
-    (fp_text value "10k" (at 4.4 0.4 unlocked) (layer "F.SilkS")
+    (fp_text value "22k" (at 4.4 0.4 unlocked) (layer "F.SilkS")
         (effects (font (size 0.75 0.75) (thickness 0.15)))
     )
@@
       (stroke (width 0.05) (type solid)) (layer "F.CrtYd"))
     (pad "1" thru_hole circle (at 0 0 270) (size 1.4 1.4) (drill 0.7) (layers "*.Cu" "*.Mask")
-      (net 33 "Net-(R43-Pad2)") (pintype "passive"))
+      (net 15 "Net-(D6-A)") (pintype "passive"))
     (pad "2" thru_hole oval (at 7.62 0 270) (size 1.4 1.4) (drill 0.7) (layers "*.Cu" "*.Mask")
       (net 35 "Net-(U2B--)") (pintype "passive"))
@@
         (effects (font (size 0.5 0.5) (thickness 0.125)))
     )
-    (fp_text value "100k" (at 4.4 0.4 -90 unlocked) (layer "F.SilkS")
+    (fp_text value "120k" (at 4.4 0.4 -90 unlocked) (layer "F.SilkS")
         (effects (font (size 0.75 0.75) (thickness 0.15)))
     )
@@
         (effects (font (size 0.5 0.5) (thickness 0.125)))
     )
-    (fp_text value "10k" (at 4.4 0.4 180 unlocked) (layer "F.SilkS")
+    (fp_text value "22k" (at 4.4 0.4 180 unlocked) (layer "F.SilkS")
         (effects (font (size 0.75 0.75) (thickness 0.15)))
     )
@@
         (effects (font (size 0.5 0.5) (thickness 0.125)))
     )
-    (fp_text value "100k" (at 4.4 0.4 -90 unlocked) (layer "F.SilkS")
+    (fp_text value "120k" (at 4.4 0.4 -90 unlocked) (layer "F.SilkS")
         (effects (font (size 0.75 0.75) (thickness 0.15)))
     )
@@
   (segment (start 184.5 121.475) (end 184.5 124.015) (width 0.25) (layer "B.Cu") (net 12))
   (segment (start 189.58 43.942) (end 187.08 46.442) (width 0.25) (layer "B.Cu") (net 13))
+  (segment (start 198 42) (end 191.5 42) (width 0.25) (layer "B.Cu") (net 13))
+  (segment (start 189.58 43.92) (end 189.58 43.942) (width 0.25) (layer "B.Cu") (net 13))
+  (segment (start 199.74 51.625) (end 199.74 43.74) (width 0.25) (layer "B.Cu") (net 13))
   (segment (start 187.08 46.442) (end 187.08 46.7) (width 0.25) (layer "B.Cu") (net 13))
+  (segment (start 199.735 51.62) (end 199.74 51.625) (width 0.25) (layer "B.Cu") (net 13))
+  (segment (start 199.74 43.74) (end 198 42) (width 0.25) (layer "B.Cu") (net 13))
+  (segment (start 191.5 42) (end 189.58 43.92) (width 0.25) (layer "B.Cu") (net 13))
   (segment (start 157.925 146.925) (end 160.1 149.1) (width 0.25) (layer "B.Cu") (net 14))
   (segment (start 157.925 141.69) (end 157.925 146.925) (width 0.25) (layer "B.Cu") (net 14))
   (segment (start 160.1 149.1) (end 176.99 149.1) (width 0.25) (layer "B.Cu") (net 14))
+  (segment (start 161.5 42.9) (end 159.1 45.3) (width 0.25) (layer "B.Cu") (net 15))
+  (segment (start 169.3 42.9) (end 161.5 42.9) (width 0.25) (layer "B.Cu") (net 15))
+  (segment (start 171.8 45.4) (end 169.3 42.9) (width 0.25) (layer "B.Cu") (net 15))
+  (segment (start 159.1 45.3) (end 159.1 51.625) (width 0.25) (layer "B.Cu") (net 15))
   (segment (start 171.8 45.4) (end 171.8 48.3) (width 0.25) (layer "B.Cu") (net 15))
   (segment (start 206.99 119.1) (end 206.9 119.1) (width 0.25) (layer "B.Cu") (net 16))
@@
   (segment (start 161.645 54.16) (end 161.64 54.165) (width 0.25) (layer "B.Cu") (net 27))
   (segment (start 161.64 54.165) (end 156.56 54.165) (width 0.25) (layer "B.Cu") (net 27))
-  (segment (start 194.67 51.62) (end 197.195 51.62) (width 0.25) (layer "B.Cu") (net 28))
-  (segment (start 197.195 51.62) (end 199.735 51.62) (width 0.25) (layer "B.Cu") (net 28))
-  (segment (start 197.2 51.615) (end 197.195 51.62) (width 0.25) (layer "B.Cu") (net 28))
-  (segment (start 197.2 46.545) (end 197.2 51.615) (width 0.25) (layer "B.Cu") (net 28))
+  (segment (start 197.2 49.195) (end 197.2 46.545) (width 0.25) (layer "B.Cu") (net 28))
   (segment (start 197.2 46.545) (end 197.2 43.942) (width 0.25) (layer "B.Cu") (net 28))
-  (segment (start 199.735 51.62) (end 199.74 51.625) (width 0.25) (layer "B.Cu") (net 28))
+  (segment (start 194.775 51.62) (end 197.2 49.195) (width 0.25) (layer "B.Cu") (net 28))
+  (segment (start 194.67 51.62) (end 194.775 51.62) (width 0.25) (layer "B.Cu") (net 28))
   (segment (start 181.96 44.005) (end 184.5 46.545) (width 0.25) (layer "B.Cu") (net 29))
   (segment (start 184.5 49.07) (end 187.05 51.62) (width 0.25) (layer "B.Cu") (net 29))
@@
   (segment (start 146.99 119.1) (end 146.99 121.39) (width 0.25) (layer "B.Cu") (net 32))
   (segment (start 157.925 129.125) (end 157.925 139.15) (width 0.25) (layer "B.Cu") (net 32))
+  (segment (start 161.64 50.14) (end 161.64 46.545) (width 0.25) (layer "B.Cu") (net 33))
   (segment (start 164.185 51.625) (end 164.19 51.62) (width 0.25) (layer "B.Cu") (net 33))
   (segment (start 164.18 45.4) (end 162.785 45.4) (width 0.25) (layer "B.Cu") (net 33))
-  (segment (start 161.64 46.545) (end 161.64 51.625) (width 0.25) (layer "B.Cu") (net 33))
-  (segment (start 159.1 51.625) (end 161.64 51.625) (width 0.25) (layer "B.Cu") (net 33))
+  (segment (start 163.12 51.62) (end 161.64 50.14) (width 0.25) (layer "B.Cu") (net 33))
   (segment (start 162.785 45.4) (end 161.64 46.545) (width 0.25) (layer "B.Cu") (net 33))
-  (segment (start 161.64 51.625) (end 164.185 51.625) (width 0.25) (layer "B.Cu") (net 33))
+  (segment (start 164.19 51.62) (end 163.12 51.62) (width 0.25) (layer "B.Cu") (net 33))
   (segment (start 197.195 64.32) (end 197.2 64.325) (width 0.25) (layer "B.Cu") (net 34))
   (segment (start 199.74 59.245) (end 197.2 61.785) (width 0.25) (layer "B.Cu") (net 34))
